File: 2025_rover_CAN_board.kicad_pcb (KiCad board)
At the start: 4 copper layers, 89.7 x 45 mm, 71 parts, among them J1 Conn_01x03, J2 Conn_01x03, J3 Conn_01x03, J4 EDIF-4, J5 RJ45 (shielded), J6 Conn_01x03, J7 Conn_01x03, SW1 SW_Push, U1 TPD4E05U06DQAR, U13 STM32G030C8T6TR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

Commit message: Add files via upload
Parts:
- J5: value RJ45 (shielded) -> R-RJ45S08P-B000; footprint Connector_RJ:RJ45_RCH_RC01937 -> footprints5:RJ45S08P-B000
- moved R20 11.0 mm to (145.5, 63.9)
- moved R21 10.9 mm to (143.0, 63.9)
- moved TP1 8.63 mm to (112.5, 56.0)
- moved TP2 8.11 mm to (128.0, 56.5)
- moved J5 7.75 mm to (95.2, 79.4), turned to 90 degrees
- moved LD2 4.34 mm to (141.0, 63.8), turned to -90 degrees
- moved LD1 4.33 mm to (139.0, 63.8), turned to -90 degrees
- moved C19 1.08 mm to (145.8, 85.2)
- moved C20 1.08 mm to (147.8, 85.2)
- moved Y2 1.08 mm to (146.7, 87.4)
Connections:
- net /CAN_H renamed /CAN_+
- net /CAN_L renamed /CAN_-
Routing:
- net /3.3V: track 14.4 -> 110.2 mm
- net GND: track 16.5 -> 72.5 mm, vias 9 -> 53
- net /5V: track 3.42 -> 51.3 mm, vias 0 -> 2
- net /16V: track 0.00 -> 45.2 mm
- net /M4_DIR: track 6.56 -> 51.7 mm, vias 2 -> 3
- net /SWCLK: track 0.00 -> 25.6 mm, vias 0 -> 2
- net /CAN_-: track 0.00 -> 24.6 mm
- net /CAN_+: track 0.00 -> 24.2 mm
- net /SWDIO: track 0.00 -> 23.9 mm, vias 0 -> 2
- net Net-(JP1-A): track 0.00 -> 22.8 mm
- net /M4_PWM: track 21.4 -> 38.6 mm
- net Net-(JP6-A): track 0.00 -> 14.5 mm
- net /M3_DIR: track 14.9 -> 28.7 mm, vias 2 -> 3
- net Net-(U3-TXCAN): track 24.8 -> 12.1 mm, vias 0 -> 2
- net /M3_PWM: track 23.8 -> 35.7 mm
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